Commit message: better model with new kinematic chain

File: iiwa_description/urdf/iiwa7.xacro (robot description, xacro)
@@ -21,22 +21,13 @@
     </joint>
     <link name="${robot_name}_link_0">
-      <inertial>
-        <origin xyz="-0.1 0 0.07" rpy="0 0 0"/>
-        <mass value="5"/>
-        <inertia ixx="0.05"  ixy="0"  ixz="0" iyy="0.06" iyz="0" izz="0.03" />
-      </inertial>
-      <visual>
-        <origin xyz="0 0 0" rpy="0 0 0"/>
-        <geometry>
-          <mesh filename="package://iiwa_description/meshes/iiwa7/visual/link_0.stl"/>
-        </geometry>
-        <material name="Grey"/>
-      </visual>
-      <collision>
-        <origin xyz="0 0 0" rpy="0 0 0"/>
-        <geometry>
-          <mesh filename="package://iiwa_description/meshes/iiwa7/collision/link_0.stl"/>
-        </geometry>
-        <material name="Grey"/>
+      <visual>
+        <geometry>
+          <mesh filename="package://iiwa_description/meshes/iiwa7/visual/base.dae"/>
+        </geometry>
+      </visual>
+      <collision>
+        <geometry>
+          <mesh filename="package://iiwa_description/meshes/iiwa7/collision/base.stl"/>
+        </geometry>
       </collision>
       <self_collision_checking>
@@ -51,5 +42,5 @@
       <parent link="${robot_name}_link_0"/>
       <child link="${robot_name}_link_1"/>
-      <origin xyz="0 0 0.15" rpy="0 0 0"/>
+      <origin xyz="0 0 0.157" rpy="0 0 0"/>
       <axis xyz="0 0 1"/>
       <limit lower="${-170 * PI / 180}" upper="${170 * PI / 180}"
@@ -62,22 +53,13 @@
     </joint>
     <link name="${robot_name}_link_1">
-      <inertial>
-        <origin xyz="0 -0.03 0.12" rpy="0 0 0"/>
-        <mass value="3.4525"/>
-        <inertia ixx="0.02183"  ixy="0"  ixz="0" iyy="0.007703" iyz="-0.003887" izz="0.02083" />
-      </inertial>
-      <visual>
-        <origin xyz="0 0 0.0075" rpy="0 0 0"/>
-        <geometry>
-          <mesh filename="package://iiwa_description/meshes/iiwa7/visual/link_1.stl"/>
-        </geometry>
-        <material name="Orange"/>
-      </visual>
-      <collision>
-        <origin xyz="0 0 0.0075" rpy="0 0 0"/>
-        <geometry>
-          <mesh filename="package://iiwa_description/meshes/iiwa7/collision/link_1.stl"/>
-        </geometry>
-        <material name="Orange"/>
+      <visual>
+        <geometry>
+          <mesh filename="package://iiwa_description/meshes/iiwa7/visual/link1.dae"/>
+        </geometry>
+      </visual>
+      <collision>
+        <geometry>
+          <mesh filename="package://iiwa_description/meshes/iiwa7/collision/link1.stl"/>
+        </geometry>
       </collision>
     </link>
@@ -85,6 +67,6 @@
       <parent link="${robot_name}_link_1"/>
       <child link="${robot_name}_link_2"/>
-      <origin xyz="0 0 0.19" rpy="${PI / 2}   0 ${PI}"/>
-      <axis xyz="0 0 1"/>
+      <origin xyz="0 0 0.183" rpy="0 0 0"/>
+      <axis xyz="0 1 0"/>
       <limit lower="${-120 * PI / 180}" upper="${120 * PI / 180}"
              effort="${max_effort}" velocity="${98 * PI / 180}" />
@@ -96,22 +78,13 @@
     </joint>
     <link name="${robot_name}_link_2">
-      <inertial>
-        <origin xyz="0.0003 0.059 0.042" rpy="0 0 0"/>
-        <mass value="3.4821"/>
-        <inertia ixx="0.02076"  ixy="0"  ixz="-0.003626" iyy="0.02179" iyz="0" izz="0.00779" />
-      </inertial>
-      <visual>
-        <origin xyz="0 0 0" rpy="0 0 0"/>
-        <geometry>
-          <mesh filename="package://iiwa_description/meshes/iiwa7/visual/link_2.stl"/>
-        </geometry>
-        <material name="Orange"/>
-      </visual>
-      <collision>
-        <origin xyz="0 0 0" rpy="0 0 0"/>
-        <geometry>
-          <mesh filename="package://iiwa_description/meshes/iiwa7/collision/link_2.stl"/>
-        </geometry>
-        <material name="Orange"/>
+      <visual>
+        <geometry>
+          <mesh filename="package://iiwa_description/meshes/iiwa7/visual/link2.dae"/>
+        </geometry>
+      </visual>
+      <collision>
+        <geometry>
+          <mesh filename="package://iiwa_description/meshes/iiwa7/collision/link2.stl"/>
+        </geometry>
       </collision>
     </link>
@@ -119,5 +92,5 @@
       <parent link="${robot_name}_link_2"/>
       <child link="${robot_name}_link_3"/>
-      <origin xyz="0 0.21 0" rpy="${PI / 2} 0 ${PI}"/>
+      <origin xyz="0 0 0.185" rpy="0 0 0"/>
       <axis xyz="0 0 1"/>
       <limit lower="${-170 * PI / 180}" upper="${170 * PI / 180}"
@@ -130,22 +103,13 @@
     </joint>
     <link name="${robot_name}_link_3">
-      <inertial>
-        <origin xyz="0 0.03 0.13" rpy="0 0 0"/>
-        <mass value="4.05623"/>
-        <inertia ixx="0.03204"  ixy="0"  ixz="0" iyy="0.00972" iyz="0.006227" izz="0.03042" />
-      </inertial>
-      <visual>
-        <origin xyz="0 0 -0.026" rpy="0 0 0"/>
-        <geometry>
-          <mesh filename="package://iiwa_description/meshes/iiwa7/visual/link_3.stl"/>
-        </geometry>
-        <material name="Orange"/>
-      </visual>
-      <collision>
-        <origin xyz="0 0 -0.026" rpy="0 0 0"/>
-        <geometry>
-          <mesh filename="package://iiwa_description/meshes/iiwa7/collision/link_3.stl"/>
-        </geometry>
-        <material name="Orange"/>
+      <visual>
+        <geometry>
+          <mesh filename="package://iiwa_description/meshes/iiwa7/visual/link3.dae"/>
+        </geometry>
+      </visual>
+      <collision>
+        <geometry>
+          <mesh filename="package://iiwa_description/meshes/iiwa7/collision/link3.stl"/>
+        </geometry>
       </collision>
     </link>
@@ -153,6 +117,6 @@
       <parent link="${robot_name}_link_3"/>
       <child link="${robot_name}_link_4"/>
-      <origin xyz="0 0 0.19" rpy="${PI / 2} 0 0"/>
-      <axis xyz="0 0 1"/>
+      <origin xyz="0 0 0.215" rpy="0 0 0"/>
+      <axis xyz="0 -1 0"/>
       <limit lower="${-120 * PI / 180}" upper="${120 * PI / 180}"
              effort="${max_effort}" velocity="${130 * PI / 180}" />
@@ -164,22 +128,13 @@
     </joint>
     <link name="${robot_name}_link_4">
-      <inertial>
-        <origin xyz="0 0.067 0.034" rpy="0 0 0"/>
-        <mass value="3.4822"/>
-        <inertia ixx="0.02178"  ixy="0"  ixz="0" iyy="0.02075" iyz="-0.003625" izz="0.007785" />
-      </inertial>
-      <visual>
-        <origin xyz="0 0 0" rpy="0 0 0"/>
-        <geometry>
-          <mesh filename="package://iiwa_description/meshes/iiwa7/visual/link_4.stl"/>
-        </geometry>
-        <material name="Orange"/>
-      </visual>
-      <collision>
-        <origin xyz="0 0 0" rpy="0 0 0"/>
-        <geometry>
-          <mesh filename="package://iiwa_description/meshes/iiwa7/collision/link_4.stl"/>
-        </geometry>
-        <material name="Orange"/>
+      <visual>
+        <geometry>
+          <mesh filename="package://iiwa_description/meshes/iiwa7/visual/link4.dae"/>
+        </geometry>
+      </visual>
+      <collision>
+        <geometry>
+          <mesh filename="package://iiwa_description/meshes/iiwa7/collision/link4.stl"/>
+        </geometry>
       </collision>
     </link>
@@ -187,5 +142,5 @@
       <parent link="${robot_name}_link_4"/>
       <child link="${robot_name}_link_5"/>
-      <origin xyz="0 0.21 0" rpy="${-PI / 2} ${PI} 0"/>
+      <origin xyz="0 0 0.4" rpy="0 0 0"/>
       <axis xyz="0 0 1"/>
       <limit lower="${-170 * PI / 180}" upper="${170 * PI / 180}"
@@ -198,22 +153,13 @@
     </joint>
     <link name="${robot_name}_link_5">
-      <inertial>
-        <origin xyz="0.0001 0.021 0.076" rpy="0 0 0"/>
-        <mass value="2.1633"/>
-        <inertia ixx="0.01287"  ixy="0"  ixz="0" iyy="0.005708" iyz="-0.003946" izz="0.01112" />
-      </inertial>
-      <visual>
-        <origin xyz="0 0 -0.026" rpy="0 0 0"/>
-        <geometry>
-          <mesh filename="package://iiwa_description/meshes/iiwa7/visual/link_5.stl"/>
-        </geometry>
-        <material name="Orange"/>
-      </visual>
-      <collision>
-        <origin xyz="0 0 -0.026" rpy="0 0 0"/>
-        <geometry>
-          <mesh filename="package://iiwa_description/meshes/iiwa7/collision/link_5.stl"/>
-        </geometry>
-        <material name="Orange"/>
+      <visual>
+        <geometry>
+          <mesh filename="package://iiwa_description/meshes/iiwa7/visual/link5.dae"/>
+        </geometry>
+      </visual>
+      <collision>
+        <geometry>
+          <mesh filename="package://iiwa_description/meshes/iiwa7/collision/link5.stl"/>
+        </geometry>
       </collision>
     </link>
@@ -221,6 +167,6 @@
       <parent link="${robot_name}_link_5"/>
       <child link="${robot_name}_link_6"/>
-      <origin xyz="0 0.06070 0.19" rpy="${PI / 2} 0 0"/>
-      <axis xyz="0 0 1"/>
+      <origin xyz="0 0 0" rpy="0 0 0"/>
+      <axis xyz="0 1 0"/>
       <limit lower="${-120 * PI / 180}" upper="${120 * PI / 180}"
              effort="${max_effort}" velocity="${180 * PI / 180}" />
@@ -232,22 +178,13 @@
     </joint>
     <link name="${robot_name}_link_6">
-      <inertial>
-        <origin xyz="0 0.0006 0.0004" rpy="0 0 0"/>
-        <mass value="2.3466"/>
-        <inertia ixx="0.006509"  ixy="0"  ixz="0" iyy="0.006259" iyz="0.00031891" izz="0.004527" />
-      </inertial>
-      <visual>
-        <origin xyz="0 0 0" rpy="0 0 0"/>
-        <geometry>
-          <mesh filename="package://iiwa_description/meshes/iiwa7/visual/link_6.stl"/>
-        </geometry>
-        <material name="Orange"/>
-      </visual>
-      <collision>
-        <origin xyz="0 0 0" rpy="0 0 0"/>
-        <geometry>
-          <mesh filename="package://iiwa_description/meshes/iiwa7/collision/link_6.stl"/>
-        </geometry>
-        <material name="Orange"/>
+      <visual>
+        <geometry>
+          <mesh filename="package://iiwa_description/meshes/iiwa7/visual/link6.dae"/>
+        </geometry>
+      </visual>
+      <collision>
+        <geometry>
+          <mesh filename="package://iiwa_description/meshes/iiwa7/collision/link6.stl"/>
+        </geometry>
       </collision>
     </link>
@@ -255,5 +192,5 @@
       <parent link="${robot_name}_link_6"/>
       <child link="${robot_name}_link_7"/>
-      <origin xyz="0 0.081 0.06070" rpy="${- PI / 2} ${PI} 0"/>
+      <origin xyz="0 0 0" rpy="0 0 0"/>
       <axis xyz="0 0 1"/>
       <limit lower="${-175 * PI / 180}" upper="${175 * PI / 180}"
@@ -266,22 +203,13 @@
     </joint>
     <link name="${robot_name}_link_7">
-      <inertial>
-        <origin xyz="0 0 0.02" rpy="0 0 0"/>
-        <mass value="3.129"/>
-        <inertia ixx="0.01464"  ixy="0.0005912"  ixz="0" iyy="0.01465" iyz="0" izz="0.002872" />
-      </inertial>
-      <visual>
-        <origin xyz="0 0 -0.0005" rpy="0 0 0"/>
-        <geometry>
-          <mesh filename="package://iiwa_description/meshes/iiwa7/visual/link_7.stl"/>
-        </geometry>
-        <material name="Grey"/>
-      </visual>
-      <collision>
-        <origin xyz="0 0 -0.0005" rpy="0 0 0"/>
-        <geometry>
-          <mesh filename="package://iiwa_description/meshes/iiwa7/collision/link_7.stl"/>
-        </geometry>
-        <material name="Grey"/>
+      <visual>
+        <geometry>
+          <mesh filename="package://iiwa_description/meshes/iiwa7/visual/link7.dae"/>
+        </geometry>
+      </visual>
+      <collision>
+        <geometry>
+          <mesh filename="package://iiwa_description/meshes/iiwa7/collision/link7.stl"/>
+        </geometry>
       </collision>
     </link>
@@ -289,5 +217,5 @@
       <parent link="${robot_name}_link_7"/>
       <child link="${robot_name}_link_ee"/>
-      <origin xyz="0 0 0.045" rpy="0 0 0"/>
+      <origin xyz="0 0 0.126" rpy="0 0 0"/>
     </joint>
     <link name="${robot_name}_link_ee">

Commit message: description: readd inertial values
Signed-off-by: Wolfgang Wiedmeyer <wolfgang.wiedmeyer@kit.edu>

File: iiwa_description/urdf/iiwa7.xacro (robot description, xacro)
@@ -21,4 +21,9 @@
     </joint>
     <link name="${robot_name}_link_0">
+      <inertial>
+        <origin xyz="-0.1 0 0.07" rpy="0 0 0"/>
+        <mass value="5"/>
+        <inertia ixx="0.05"  ixy="0"  ixz="0" iyy="0.06" iyz="0" izz="0.03" />
+      </inertial>
       <visual>
         <geometry>
@@ -53,4 +58,9 @@
     </joint>
     <link name="${robot_name}_link_1">
+      <inertial>
+        <origin xyz="0 -0.03 0.12" rpy="0 0 0"/>
+        <mass value="3.4525"/>
+        <inertia ixx="0.02183"  ixy="0"  ixz="0" iyy="0.007703" iyz="-0.003887" izz="0.02083" />
+      </inertial>
       <visual>
         <geometry>
@@ -78,4 +88,9 @@
     </joint>
     <link name="${robot_name}_link_2">
+      <inertial>
+        <origin xyz="0.0003 0.059 0.042" rpy="0 0 0"/>
+        <mass value="3.4821"/>
+        <inertia ixx="0.02076"  ixy="0"  ixz="-0.003626" iyy="0.02179" iyz="0" izz="0.00779" />
+      </inertial>
       <visual>
         <geometry>
@@ -103,4 +118,9 @@
     </joint>
     <link name="${robot_name}_link_3">
+      <inertial>
+        <origin xyz="0 0.03 0.13" rpy="0 0 0"/>
+        <mass value="4.05623"/>
+        <inertia ixx="0.03204"  ixy="0"  ixz="0" iyy="0.00972" iyz="0.006227" izz="0.03042" />
+      </inertial>
       <visual>
         <geometry>
@@ -128,4 +148,9 @@
     </joint>
     <link name="${robot_name}_link_4">
+      <inertial>
+        <origin xyz="0 0.067 0.034" rpy="0 0 0"/>
+        <mass value="3.4822"/>
+        <inertia ixx="0.02178"  ixy="0"  ixz="0" iyy="0.02075" iyz="-0.003625" izz="0.007785" />
+      </inertial>
       <visual>
         <geometry>
@@ -153,4 +178,9 @@
     </joint>
     <link name="${robot_name}_link_5">
+      <inertial>
+        <origin xyz="0.0001 0.021 0.076" rpy="0 0 0"/>
+        <mass value="2.1633"/>
+        <inertia ixx="0.01287"  ixy="0"  ixz="0" iyy="0.005708" iyz="-0.003946" izz="0.01112" />
+      </inertial>
       <visual>
         <geometry>
@@ -178,4 +208,9 @@
     </joint>
     <link name="${robot_name}_link_6">
+      <inertial>
+        <origin xyz="0 0.0006 0.0004" rpy="0 0 0"/>
+        <mass value="2.3466"/>
+        <inertia ixx="0.006509"  ixy="0"  ixz="0" iyy="0.006259" iyz="0.00031891" izz="0.004527" />
+      </inertial>
       <visual>
         <geometry>
@@ -203,4 +238,9 @@
     </joint>
     <link name="${robot_name}_link_7">
+      <inertial>
+        <origin xyz="0 0 0.02" rpy="0 0 0"/>
+        <mass value="3.129"/>
+        <inertia ixx="0.01464"  ixy="0.0005912"  ixz="0" iyy="0.01465" iyz="0" izz="0.002872" />
+      </inertial>
       <visual>
         <geometry>
